File: PCB/HogwartsFlasksMain.sch (KiCad schematic (older format))
At the start: 186 parts, among them Q1 IRLML6401, U1 USBLC6

Commit message: PCB Layout done
Parts:
- removed TP1, TP2: TESTPOINT, PCB:TESTPOINT_1d5MM, symbol pcb_details:TESTPOINT
- C40, C41, C43, C44, C51, C55: footprint Capacitors:CAP_0603 -> Capacitors:CAP_0402
- Logo1: footprint Pictures:Ostranna_16d9_13d5 -> Pictures:Ostranna_12d7_10d1
Connections:
- net GND_IN is gone; now on net GND: C4.2
- net GND: now also XL9.1, XL9.2
Changed lines of the file:
@@
 	1    0    0    -1
 $EndComp
-$Comp
-L pcb_details:TESTPOINT TP1
-U 1 1 5D688A3A
-P 1300 14050
-F 0 "TP1" H 1256 14156 60  0000 C CNN
-F 1 "TESTPOINT" H 1275 14275 60  0001 C CNN
-F 2 "PCB:TESTPOINT_1d5MM" H 1200 14100 60  0001 C CNN
-F 3 "" H 1300 14200 60  0001 C CNN
-F 4 "0" H 1400 14300 60  0001 C CNN "Price"
-F 5 "0" H 1500 14400 60  0001 C CNN "SolderPoints"
-	1    1300 14050
-	1    0    0    -1
-$EndComp
-$Comp
-L pcb_details:TESTPOINT TP2
-U 1 1 5D688A3B
-P 1450 15050
-F 0 "TP2" V 1407 14997 60  0000 R CNN
-F 1 "TESTPOINT" H 1425 15275 60  0001 C CNN
-F 2 "PCB:TESTPOINT_1d5MM" H 1350 15100 60  0001 C CNN
-F 3 "" H 1450 15200 60  0001 C CNN
-F 4 "0" H 1550 15300 60  0001 C CNN "Price"
-F 5 "0" H 1650 15400 60  0001 C CNN "SolderPoints"
-	1    1450 15050
-	0    -1   -1   0
-$EndComp
 Wire Wire Line
 	850  15050 1150 15050
@@
 	1450 14850 1450 14650
 Wire Wire Line
-	1450 13000 1900 13000
-Wire Wire Line
 	1450 13950 1450 14050
-Wire Wire Line
-	1300 14050 1450 14050
-Wire Wire Line
-	1450 15050 1450 14850
-Text Label 1900 13000 2    60   ~ 0
-GND_IN
-Connection ~ 1450 14850
 Text Label 2600 14050 2    60   ~ 0
 5V_USB
@@
 	1    0    0    -1
 $EndComp
-$Comp
-L Tittar_kl:C C55
-U 1 1 5D6A2135
-P 14550 3550
-F 0 "C55" H 14450 3450 50  0000 L CNN
-F 1 "0.1u" H 14450 3650 50  0000 L CNN
-F 2 "Capacitors:CAP_0603" V 14650 3400 28  0001 C BNN
-F 3 "" H 14550 3550 60  0001 C CNN
-	1    14550 3550
-	1    0    0    -1
-$EndComp
 Wire Wire Line
 	14850 3300 14550 3300
@@
 F 0 "C51" H 14200 3450 50  0000 L CNN
 F 1 "0.1u" H 14200 3650 50  0000 L CNN
-F 2 "Capacitors:CAP_0603" V 14400 3400 28  0001 C BNN
+F 2 "Capacitors:CAP_0402" V 14400 3400 28  0001 C BNN
 F 3 "" H 14300 3550 60  0001 C CNN
 	1    14300 3550
@@
 F 0 "C44" H 13950 3450 50  0000 L CNN
 F 1 "47pF" H 13950 3650 50  0000 L CNN
-F 2 "Capacitors:CAP_0603" V 14150 3400 28  0001 C BNN
+F 2 "Capacitors:CAP_0402" V 14150 3400 28  0001 C BNN
 F 3 "" H 14050 3550 60  0001 C CNN
 	1    14050 3550
@@
 F 0 "C41" H 13450 3450 50  0000 L CNN
 F 1 "0.1u" H 13450 3650 50  0000 L CNN
-F 2 "Capacitors:CAP_0603" V 13650 3400 28  0001 C BNN
+F 2 "Capacitors:CAP_0402" V 13650 3400 28  0001 C BNN
 F 3 "" H 13550 3550 60  0001 C CNN
 	1    13550 3550
@@
 F 0 "C40" H 13200 3450 50  0000 L CNN
 F 1 "0.1u" H 13200 3650 50  0000 L CNN
-F 2 "Capacitors:CAP_0603" V 13400 3400 28  0001 C BNN
+F 2 "Capacitors:CAP_0402" V 13400 3400 28  0001 C BNN
 F 3 "" H 13300 3550 60  0001 C CNN
 	1    13300 3550
@@
 $EndComp
 $Comp
-L Tittar_kl:L L6
-U 1 1 5D6AC2BA
-P 13700 4350
-F 0 "L6" V 13900 4350 50  0000 C CNN
-F 1 "Choke" V 13800 4350 50  0000 C CNN
-F 2 "Inductors:IND_0402" V 13760 4360 40  0001 C CNN
-F 3 "" V 13600 4210 60  0001 C CNN
-F 4 "1" V 13700 4310 60  0001 C CNN "Price"
-F 5 "2" V 13800 4410 60  0001 C CNN "SolderPoints"
-F 6 "SBY100505T-102Y-N" V 13700 4350 50  0001 C CNN "PN"
-	1    13700 4350
-	0    1    -1   0
-$EndComp
-Wire Wire Line
-	13500 4350 13400 4350
-$Comp
-L power:VCC #PWR084
-U 1 1 5D6AC76B
-P 14000 4350
-F 0 "#PWR084" H 14000 4400 30  0001 C CNN
-F 1 "VCC" H 14037 4417 30  0000 C CNN
-F 2 "" H 14000 4350 60  0000 C CNN
-F 3 "" H 14000 4350 60  0000 C CNN
-	1    14000 4350
-	1    0    0    -1
-$EndComp
-Wire Wire Line
-	14000 4350 13900 4350
-$Comp
 L Tittar_kl:L L11
 U 1 1 5D6AD032
@@
 F 0 "C43" H 13700 3450 50  0000 L CNN
 F 1 "0.1u" H 13700 3650 50  0000 L CNN
-F 2 "Capacitors:CAP_0603" V 13900 3400 28  0001 C BNN
+F 2 "Capacitors:CAP_0402" V 13900 3400 28  0001 C BNN
 F 3 "" H 13800 3550 60  0001 C CNN
 	1    13800 3550
@@
 Wire Wire Line
 	21700 2600 22050 2600
-$Comp
-L Tittar_kl:R R21
-U 1 1 5D6376A2
-P 18700 3000
-F 0 "R21" V 18780 2850 50  0000 C CNN
-F 1 "1k" V 18700 3000 50  0000 C CNN
-F 2 "Resistors:RES_0603" V 18780 3100 28  0001 C CNN
-F 3 "" V 18780 2850 60  0000 C CNN
-F 4 "0.5" V 18880 2950 60  0001 C CNN "Price"
-F 5 "2" V 18980 3050 60  0001 C CNN "SolderPoints"
-	1    18700 3000
-	0    -1   -1   0
-$EndComp
 Wire Wire Line
 	18950 3000 19150 3000
@@
 $EndComp
 $Comp
-L Audio_kl:CS42L52 DA4
-U 1 1 5D6EBE88
-P 13150 6900
-F 0 "DA4" H 13100 8637 60  0000 C CNN
-F 1 "CS42L52" H 13100 8531 60  0000 C CNN
-F 2 "QFN_DFN:QFN40" H 13150 7150 60  0001 C CNN
-F 3 "" H 13150 7150 60  0001 C CNN
-F 4 "41" H 12650 8600 60  0001 C CNN "SolderPoints"
-F 5 "61" H 13150 6900 60  0001 C CNN "Price"
-	1    13150 6900
-	1    0    0    -1
-$EndComp
-$Comp
 L Tittar_kl:C C57
 U 1 1 5D6EBE89
@@
 $EndComp
 $Comp
-L Tittar_kl:C C56
-U 1 1 5D6EBE91
-P 14550 7150
-F 0 "C56" H 14550 7250 50  0000 L CNN
-F 1 "1u" H 14550 7050 50  0000 L CNN
-F 2 "Capacitors:CAP_0603" V 14650 7000 28  0001 C BNN
-F 3 "" H 14450 7050 60  0001 C CNN
-F 4 "0.5" H 14550 7150 60  0001 C CNN "Price"
-F 5 "2" H 14650 7250 60  0001 C CNN "SolderPoints"
-	1    14550 7150
-	1    0    0    -1
-$EndComp
-$Comp
 L power:GND #PWR095
 U 1 1 5D6EBE92
@@
 F 0 "Logo1" H 22450 13950 60  0000 C CNN
 F 1 "Logo" H 22750 13950 60  0000 C CNN
-F 2 "Pictures:Ostranna_16d9_13d5" H 22550 13500 60  0001 C CNN
+F 2 "Pictures:Ostranna_12d7_10d1" H 22550 13500 60  0001 C CNN
 F 3 "" H 22550 13500 60  0000 C CNN
 	1    22550 13500
@@
 Text Notes 12000 12800 2    100  ~ 20
 Power\n
+$Comp
+L Tittar_kl:R R21
+U 1 1 5D6376A2
+P 18700 3000
+F 0 "R21" V 18780 2850 50  0000 C CNN
+F 1 "1k" V 18700 3000 50  0000 C CNN
+F 2 "Resistors:RES_0603" V 18780 3100 28  0001 C CNN
+F 3 "" V 18780 2850 60  0000 C CNN
+F 4 "0.5" V 18880 2950 60  0001 C CNN "Price"
+F 5 "2" V 18980 3050 60  0001 C CNN "SolderPoints"
+	1    18700 3000
+	0    -1   -1   0
+$EndComp
+$Comp
+L Tittar_kl:C C55
+U 1 1 5D6A2135
+P 14550 3550
+F 0 "C55" H 14450 3450 50  0000 L CNN
+F 1 "0.1u" H 14450 3650 50  0000 L CNN
+F 2 "Capacitors:CAP_0402" V 14650 3400 28  0001 C BNN
+F 3 "" H 14550 3550 60  0001 C CNN
+	1    14550 3550
+	1    0    0    -1
+$EndComp
+$Comp
+L power:GND #PWR0151
+U 1 1 5D919855
+P 22000 11900
+F 0 "#PWR0151" H 22090 11880 30  0001 C CNN
+F 1 "GND" H 22000 11820 30  0001 C CNN
+F 2 "" H 22000 11900 60  0000 C CNN
+F 3 "" H 22000 11900 60  0000 C CNN
+	1    22000 11900
+	1    0    0    -1
+$EndComp
+$Comp
+L Audio_kl:CS42L52 DA4
+U 1 1 5D6EBE88
+P 13150 6900
+F 0 "DA4" H 13100 8637 60  0000 C CNN
+F 1 "CS42L52" H 13100 8531 60  0000 C CNN
+F 2 "QFN_DFN:QFN40" H 13150 7150 60  0001 C CNN
+F 3 "" H 13150 7150 60  0001 C CNN
+F 4 "41" H 12650 8600 60  0001 C CNN "SolderPoints"
+F 5 "61" H 13150 6900 60  0001 C CNN "Price"
+	1    13150 6900
+	1    0    0    -1
+$EndComp
+$Comp
+L power:VCC #PWR084
+U 1 1 5D6AC76B
+P 14050 4350
+F 0 "#PWR084" H 14050 4400 30  0001 C CNN
+F 1 "VCC" H 14087 4417 30  0000 C CNN
+F 2 "" H 14050 4350 60  0000 C CNN
+F 3 "" H 14050 4350 60  0000 C CNN
+	1    14050 4350
+	1    0    0    -1
+$EndComp
+$Comp
+L power:PWR_FLAG #FLG0103
+U 1 1 5DB93EAA
+P 13950 4250
+F 0 "#FLG0103" H 13950 4520 30  0001 C CNN
+F 1 "PWR_FLAG" H 13950 4457 30  0000 C CNN
+F 2 "" H 13950 4250 60  0000 C CNN
+F 3 "" H 13950 4250 60  0000 C CNN
+	1    13950 4250
+	1    0    0    -1
+$EndComp
+Wire Wire Line
+	13500 4350 13400 4350
+Wire Wire Line
+	14050 4350 13950 4350
+$Comp
+L Tittar_kl:L L6
+U 1 1 5D6AC2BA
+P 13700 4350
+F 0 "L6" V 13900 4350 50  0000 C CNN
+F 1 "Choke" V 13800 4350 50  0000 C CNN
+F 2 "Inductors:IND_0402" V 13760 4360 40  0001 C CNN
+F 3 "" V 13600 4210 60  0001 C CNN
+F 4 "1" V 13700 4310 60  0001 C CNN "Price"
+F 5 "2" V 13800 4410 60  0001 C CNN "SolderPoints"
+F 6 "SBY100505T-102Y-N" V 13700 4350 50  0001 C CNN "PN"
+	1    13700 4350
+	0    1    -1   0
+$EndComp
+Wire Wire Line
+	13950 4250 13950 4350
+Connection ~ 13950 4350
+Wire Wire Line
+	13950 4350 13900 4350
+$Comp
+L power:GND #PWR0152
+U 1 1 5DB9E1D9
+P 1450 12950
+F 0 "#PWR0152" H 1540 12930 30  0001 C CNN
+F 1 "GND" H 1450 12870 30  0001 C CNN
+F 2 "" H 1450 12950 60  0000 C CNN
+F 3 "" H 1450 12950 60  0000 C CNN
+	1    1450 12950
+	1    0    0    -1
+$EndComp
+Wire Wire Line
+	1450 12950 1450 13000
+$Comp
+L Tittar_kl:C C56
+U 1 1 5D6EBE91
+P 14550 7150
+F 0 "C56" H 14550 7250 50  0000 L CNN
+F 1 "1u" H 14550 7050 50  0000 L CNN
+F 2 "Capacitors:CAP_0603" V 14650 7000 28  0001 C BNN
+F 3 "" H 14450 7050 60  0001 C CNN
+F 4 "0.5" H 14550 7150 60  0001 C CNN "Price"
+F 5 "2" H 14650 7250 60  0001 C CNN "SolderPoints"
+	1    14550 7150
+	1    0    0    -1
+$EndComp
 $EndSCHEMATC

Commit message: Proceeding with tracing
Parts:
- removed R22: 33R, Resistors:RES_0603, symbol Tittar_kl:R
- removed XL9: CONN_5, Connectors:SLD_5_2D5, symbol Connectors_kl:CONN_5
- added C87: 0.1u, Capacitors:CAP_0603, symbol Tittar_kl:C
- added DA8: MC74VHC1, SOT:SOT23-5, symbol standard_logic:1xBUF_W3STATE
- added R25: 33R, Resistors:RES_0603, symbol Tittar_kl:R
- added XL10, XL9: CONN_3, Connectors:SLD_3_2D5, symbol Connectors_kl:CONN_3
Connections:
- net +5v: now also C87.1, DA8.5 (Vcc), XL10.3, XL9.3
- net GND: now also C87.2, DA8.1 (~OE), DA8.3 (GND), XL10.1 (P1), XL9.1 (P1)
- net LCD_BACKLT: now also DD1.18 (PF6/T10C1/RX7/ADC3-4); no longer DD1.135 (PB5/MOSI6/MOSI3/MOSI1/T3C2/RX5)
- net NPX_CTRL: now also DA7.2 (InA)
- net at R23.1: now also XL9.2 (PM)
- new net: DA8.4 (OutY), R25.2
- new net: R25.1, XL10.2 (PM)
- new net NPX_CTRL2: DA8.2 (InA), DD1.135 (PB5/MOSI6/MOSI3/MOSI1/T3C2/RX5)
- no-connect marks 35 -> 34
Other:
- note added: "Periphery\n\nSPI1 (PB5) Neopix2 ctrl, DMA2 S5 C3\nSPI5 (PF5) Neopix ctrl, DMA2 S4 C2\n\nT10C1 (PF6) LCD BCKLT\nT11C1 (PF7) LED"
- moved on the sheet: C78, C81, DA7, HOLE1, HOLE2, HOLE3, HOLE4, Logo1, R23

Commit message: PCB sent to factory
Parts:
- C1, C10, C11, C12, C13, C15, C16, C17, C18, C19, C2, C20, C21, C22, C23, C24, C25, C26, C27, C28, C29, C3, C30, C31, C32, C33, C34, C35, C36, C37, C38, C39, C4, C42, C45, C46, C47, C48, C49, C5, C50, C52, C53, C56, C57, C58, C59, C6, C61, C63, C64, C67, C7, C70, C71, C72, C75, C77, C8, C80, C81, C85, C87, C9: footprint Capacitors:CAP_0603 -> Capacitors:CAP_0603_Silks
