File: PCB/HogwartsFlasksMain.kicad_pcb (KiCad board)
At the start: 4 copper layers, 108 x 63 mm, 184 parts, among them Q1 IRLML6401, U1 USBLC6

Commit message: Proceeding with tracing
Parts:
- removed R22: 33R, Resistors:RES_0603
- added C87: 0.1u, Capacitors:CAP_0603, F.Cu at (195.8, 95.2)
- added DA8: MC74VHC1, SOT:SOT23-5, F.Cu at (198.4, 95.2)
- added R25: 33R, Resistors:RES_0603, F.Cu at (202.0, 91.1)
- added XL10: CONN_3, Connectors:SLD_3_2D5, F.Cu at (205.8, 91.1)
- XL9: value CONN_5 -> CONN_3; footprint Connectors:SLD_5_2D5 -> Connectors:SLD_3_2D5
- moved XL9 2.98 mm to (205.8, 101.1), turned to 90 degrees
- moved R23 2.91 mm to (202.0, 101.1)
- moved C34 1.60 mm to (191.0, 87.3)
- moved C35 1.60 mm to (187.0, 80.8)
- moved C37 1.60 mm to (193.0, 90.3)
- moved C39 1.60 mm to (192.6, 87.3)
- moved C45 1.60 mm to (197.9, 75.1)
- moved C48 1.60 mm to (199.7, 77.1)
- moved C52 1.60 mm to (199.7, 81.6)
- moved C56 1.60 mm to (199.7, 83.8)
- moved DA4 1.60 mm to (193.3, 80.6)
- moved R12 1.60 mm to (189.4, 87.3)
- moved R13 1.60 mm to (194.2, 87.3)
- moved TP6 1.60 mm to (194.6, 89.6)
- moved TP7 1.60 mm to (186.3, 87.6)
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Connections:
- DA7 pad 2: Net-(DA7-Pad2) -> /NPX_CTRL
- DD1 pad 135: /LCD_BACKLT -> /NPX_CTRL2
- DD1 pad 18: (no net) -> /LCD_BACKLT
- XL9 pad 2: GND -> Net-(R23-Pad1)
- XL9 pad 3: Net-(R23-Pad1) -> +5v
Other:
- net class Default: via_dia 0.7 -> 0.6
- net class Wide: via_dia 0.7 -> 0.6

Commit message: PCB sent to factory
Parts:
- C1, C10, C11, C12, C13, C15, C16, C17, C18, C19, C2, C20, C21, C22, C23, C24, C25, C26, C27, C28, C29, C3, C30, C31, C32, C33, C34, C35, C36, C37, C38, C39, C4, C42, C45, C46, C47, C48, C49, C5, C50, C52, C53, C56, C57, C58, C59, C6, C61, C63, C64, C67, C7, C70, C71, C72, C75, C77, C8, C80, C81, C85, C87, C9: footprint Capacitors:CAP_0603 -> Capacitors:CAP_0603_Silks
- moved TP15 6.53 mm to (119.2, 97.0)
- moved TP14 5.80 mm to (117.8, 97.0)
- moved TP27 4.10 mm to (184.2, 111.0)
- moved C85 3.10 mm to (184.6, 112.6), turned to 180 degrees
- moved TP13 2.92 mm to (118.4, 95.0)
- moved TP12 1.50 mm to (121.0, 96.4)
- moved L14 1.50 mm to (185.4, 110.6)
- moved TP11 1.30 mm to (121.0, 95.0)
- moved Logo1 1.02 mm to (170.3, 67.3)
- moved C77 1.00 mm to (164.2, 90.4)
- moved C66 0.92 mm to (117.2, 86.4), turned to 180 degrees
- moved L8 0.85 mm to (181.4, 100.2), turned to 270 degrees
- moved C33 0.83 mm to (170.9, 109.9)
- moved C54 0.83 mm to (181.2, 107.9)
- moved D2 0.83 mm to (177.6, 104.2)
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Routing:
- net GND: track 0.00 -> 837.5 mm, vias 0 -> 302
- net PwrMCU: track 0.00 -> 166.7 mm, vias 0 -> 14
- net +3v3: track 0.00 -> 134.7 mm, vias 0 -> 6
- net +5v: track 0.00 -> 111.0 mm
- net /LTDC_VSYNC: track 0.00 -> 74.5 mm, vias 0 -> 2
- net /LTDC_CLK: track 0.00 -> 74.1 mm, vias 0 -> 2
- net /LTDC_HSYNC: track 0.00 -> 73.9 mm, vias 0 -> 2
- net /SCL: track 0.00 -> 72.7 mm, vias 0 -> 2
- net /LTDC_DE: track 0.00 -> 71.2 mm, vias 0 -> 2
- net /SDA: track 0.00 -> 70.9 mm, vias 0 -> 2
- net /LTDC_R0: track 0.00 -> 69.0 mm, vias 0 -> 2
- net /LTDC_B4: track 0.00 -> 68.9 mm, vias 0 -> 2
- net /AU_RST: track 0.00 -> 68.7 mm, vias 0 -> 3
- net /NPX_CTRL2: track 0.00 -> 68.6 mm, vias 0 -> 2
- net /LTDC_B5: track 0.00 -> 67.6 mm, vias 0 -> 2
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- added copper zone on B.Cu, net GND
- added copper zone on F.Cu, net GND
- added copper zone on In1.Cu, net GND
- added copper zone on In2.Cu, net GND
Other:
- board text added: "CLK"
- board text added: "DE"
- board text added: "DISP"
- board text added: "H"
- board text added: "MISO"
- board text added: "MOSI"
- board text added: "Memory"
- board text added: "NSS"
- board text added: "Ostranna Hogwarts Flasks 01"
- board text added: "SCK"
- board text added: "SD"
- board text added: "Sound"
- board text added: "V"

Commit message: Fighting w JPEG
Other:
- net class Default removed
- net class Wide removed
