File: PCB/HogwartsFlasksMain.kicad_sch (KiCad schematic)
At the start: 187 parts, among them Q1 IRLML6401, U1 USBLC6

Commit message: Working somehow
Other:
- note added: "Reality: VLED- VLED+ GND VDD"
Changed lines of the file:
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@@
   (junction (at 535.94 143.51) (diameter 0) (color 0 0 0 0))
   (junction (at 551.18 66.04) (diameter 0) (color 0 0 0 0))
+  (no_connect (at 104.14 93.98))
+  (no_connect (at 354.33 156.21))
+  (no_connect (at 104.14 144.78))
   (no_connect (at 377.19 54.61))
-  (no_connect (at 377.19 52.07))
+  (no_connect (at 416.56 54.61))
+  (no_connect (at 438.15 302.26))
+  (no_connect (at 201.93 187.96))
+  (no_connect (at 311.15 191.77))
+  (no_connect (at 416.56 52.07))
+  (no_connect (at 438.15 284.48))
+  (no_connect (at 416.56 73.66))
   (no_connect (at 558.8 234.95))
-  (no_connect (at 438.15 304.8))
-  (no_connect (at 416.56 54.61))
-  (no_connect (at 311.15 189.23))
-  (no_connect (at 104.14 167.64))
-  (no_connect (at 438.15 302.26))
-  (no_connect (at 558.8 222.25))
-  (no_connect (at 104.14 93.98))
-  (no_connect (at 558.8 227.33))
-  (no_connect (at 311.15 179.07))
-  (no_connect (at 354.33 156.21))
+  (no_connect (at 558.8 232.41))
+  (no_connect (at 311.15 181.61))
   (no_connect (at 311.15 186.69))
   (no_connect (at 311.15 184.15))
+  (no_connect (at 24.13 379.73))
+  (no_connect (at 558.8 229.87))
+  (no_connect (at 558.8 227.33))
+  (no_connect (at 438.15 281.94))
+  (no_connect (at 377.19 52.07))
+  (no_connect (at 311.15 189.23))
+  (no_connect (at 311.15 173.99))
+  (no_connect (at 311.15 196.85))
+  (no_connect (at 311.15 179.07))
   (no_connect (at 201.93 115.57))
-  (no_connect (at 311.15 181.61))
-  (no_connect (at 416.56 73.66))
+  (no_connect (at 311.15 158.75))
+  (no_connect (at 104.14 167.64))
+  (no_connect (at 438.15 304.8))
+  (no_connect (at 558.8 222.25))
+  (no_connect (at 354.33 138.43))
+  (no_connect (at 311.15 176.53))
   (no_connect (at 106.68 365.76))
   (no_connect (at 354.33 140.97))
-  (no_connect (at 416.56 52.07))
-  (no_connect (at 104.14 144.78))
-  (no_connect (at 558.8 229.87))
-  (no_connect (at 311.15 173.99))
-  (no_connect (at 558.8 232.41))
-  (no_connect (at 311.15 191.77))
-  (no_connect (at 24.13 379.73))
-  (no_connect (at 201.93 187.96))
-  (no_connect (at 311.15 196.85))
-  (no_connect (at 438.15 281.94))
-  (no_connect (at 438.15 284.48))
-  (no_connect (at 354.33 138.43))
-  (no_connect (at 311.15 176.53))
-  (no_connect (at 311.15 158.75))
   (wire (pts (xy 21.59 379.73) (xy 21.59 382.27))
     (stroke (width 0) (type solid) (color 0 0 0 0))
@@
     (effects (font (size 2.0066 2.0066) (thickness 0.4013) bold) (justify right bottom))
   )
+  (text "Reality:\nVLED-\nVLED+\nGND\nVDD" (at 580.39 142.24 180)
+    (effects (font (size 1.27 1.27)) (justify right bottom))
+  )
   (label "SD_PWR_EN" (at 21.59 316.23 0)
